File: pulseoximeter.kicad_pcb (KiCad board)
At the start: 4 copper layers, 38 x 80.1 mm, 49 parts, among them J1 X05A20L15T, J2 TYPE-C-31-M-12, J3 Conn_01x02, U1 TPD2EUSB30DRTR, U2 TPS7A4700RGWR, U3 ESP32-S3-MINI-1-N8, U4 LM324, U6 OPA140AIDBVR, U7 DMN2310UT-13

Commit message: layout complete
Parts:
- removed C18: 440pF, Capacitor_SMD:C_0603_1608Metric
- removed C6: 10uF, Capacitor_SMD:C_0603_1608Metric
- removed C7: 0.1uF, Capacitor_SMD:C_0603_1608Metric
- removed D2, D3: LED, LED_THT:LED_D3.0mm
- removed R1: 10k, Resistor_SMD:R_0402_1005Metric
- removed R14, R22: 330, Resistor_SMD:R_0603_1608Metric
- removed R2: 1M, Resistor_SMD:R_0402_1005Metric
- removed U7: DMN2310UT-13, Package_TO_SOT_SMD:SOT-523
- added C8: 22uF, Capacitor_SMD:C_0603_1608Metric, F.Cu at (141.8, 88.0)
- added D4: LED, LED_THT:LED_D3.0mm, F.Cu at (144.2, 115.2)
- added D7: LED, LED_THT:LED_D3.0mm, F.Cu at (128.0, 108.0)
- added D8: LED, LED_THT:LED_D3.0mm, F.Cu at (128.0, 112.8)
- added D9: LED, LED_THT:LED_D3.0mm, F.Cu at (160.5, 108.0)
- added TP3: TestPoint, TestPoint:TestPoint_Pad_D1.0mm, F.Cu at (138.2, 88.5)
- added TP4: TestPoint, TestPoint:TestPoint_Pad_D1.0mm, F.Cu at (156.2, 70.8)
- added U5: TLC59116IPWR, TLC59116IPWR:PW28, F.Cu at (158.5, 94.4)
- R11: value 8.1M -> 5.6M
- R13: value 330 -> 10k
- R7: value 330 -> 931
- moved R13 37.1 mm to (163.0, 87.0), turned to 90 degrees
- moved R7 32.0 mm to (158.2, 87.0), turned to -90 degrees
- moved D6 15.9 mm to (160.5, 112.8)
- moved D5 13.1 mm to (144.2, 127.2)
- moved D1 12.6 mm to (144.2, 121.2)
- moved R12 11.1 mm to (141.8, 102.8)
- moved C19 10.8 mm to (139.0, 100.2), turned to 180 degrees
- moved R11 7.24 mm to (146.0, 108.8), turned to 0 degrees
- moved U6 4.81 mm to (146.0, 104.5), turned to 0 degrees
- moved C1 3.78 mm to (132.5, 89.2), turned to 180 degrees
- moved C13 2.31 mm to (149.8, 108.8)
- moved R10 2.25 mm to (149.0, 95.0)
- moved R6 2.25 mm to (152.8, 85.2)
- moved R9 2.25 mm to (149.0, 91.5)
- moved R23 1.49 mm to (136.0, 97.3)
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Connections:
- D5 pad 1: GND -> Net-(D5-K)
- D5 pad 2: Net-(D5-A) -> VBUS
- D6 pad 1: GND -> Net-(D6-K)
- D6 pad 2: Net-(D6-A) -> VBUS
- R10 pad 1: Net-(U4D--) -> Net-(U4D-+)
- R13 pad 1: VBUS -> Net-(U5-*RESET)
- R13 pad 2: Net-(D6-A) -> +3.3V
- R7 pad 1: VBUS -> GND
- R7 pad 2: Net-(D5-A) -> Net-(U5-REXT)
- R9 pad 2: Net-(U4D--) -> Net-(U4D-+)
- U3 pad 16: /DISPLAY_D/C -> /TP_INT
- U3 pad 17: /DISPLAY_CS -> /TP_RST
- U3 pad 18: /DISPLAY_CLK -> /DISPLAY_RESET
- U3 pad 20: /DISPLAY_RESET -> /DISPLAY_CLK
- U3 pad 21: /TP_RST -> /DISPLAY_CS
- U3 pad 22: /TP_INT -> /DISPLAY_D/C
- U4 pad 12: VCC/2 -> Net-(U4D-+)
- U4 pad 13: Net-(U4D--) -> VCC/2
- U4 pad 4: VBUS -> +3.3V
- U6 pad 5: VBUS -> +3.3V
Routing:
- net VBUS: track 97.4 -> 176.3 mm, vias 6 -> 5
- net Net-(D7-K): track 0.00 -> 76.5 mm, vias 0 -> 1
- net Net-(D8-K): track 0.00 -> 74.1 mm, vias 0 -> 1
- net +3.3V: track 78.7 -> 134.1 mm, vias 4 -> 9
- net Net-(D4-K): track 0.00 -> 54.5 mm, vias 0 -> 1
- net Net-(D5-K): track 0.00 -> 38.7 mm, vias 0 -> 1
- net SDA: track 13.6 -> 43.6 mm, vias 1 -> 3
- net /LEDK: track 5.85 -> 33.6 mm, vias 0 -> 3
- net SCL: track 10.6 -> 35.0 mm, vias 1 -> 3
- net Net-(D6-K): track 0.00 -> 20.0 mm, vias 0 -> 1
- net /DISPLAY_D/C: track 0.76 -> 19.4 mm
- net /DISPLAY_CS: track 1.04 -> 19.6 mm
- net /DISPLAY_CLK: track 1.21 -> 19.7 mm
- net /DISPLAY_SDI: track 1.49 -> 19.9 mm
- net /DISPLAY_RESET: track 1.72 -> 20.0 mm
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- added copper zone on In1.Cu, net GND
Other:
- board size 38 x 80.1 mm -> 38 x 78.7 mm

Commit message: -
Parts:
- removed C8: 22uF, Capacitor_SMD:C_0603_1608Metric
- added JP1: SolderJumper_2_Bridged, Jumper:SolderJumper-2_P1.3mm_Open_RoundedPad1.0x1.5mm, F.Cu at (140.8, 103.8)
- added JP3: SolderJumper_2_Bridged, Jumper:SolderJumper-2_P1.3mm_Open_RoundedPad1.0x1.5mm, F.Cu at (151.6, 100.2)
- added R1: 100k, Resistor_SMD:R_0603_1608Metric, F.Cu at (141.8, 87.2)
- added R2: 50k, Resistor_SMD:R_0603_1608Metric, F.Cu at (139.5, 88.7)
- added TP5: TestPoint, TestPoint:TestPoint_Pad_D1.0mm, F.Cu at (152.2, 74.5)
- C13: value 0.1uF -> 0.22uF
- C3: footprint Capacitor_SMD:C_0402_1005Metric -> Capacitor_SMD:C_0603_1608Metric
- R7: value 931 -> 910
- moved C19 4.81 mm to (143.8, 101.0), turned to 0 degrees
- moved R12 2.47 mm to (140.0, 101.0), turned to 180 degrees
- moved TP3 1.06 mm to (137.5, 89.2)
- moved C20 0.75 mm to (132.5, 93.8)
- moved R10 0.75 mm to (149.0, 95.8)
- moved R23 0.75 mm to (136.0, 98.1)
- moved R24 0.75 mm to (136.0, 93.8)
- moved R9 0.75 mm to (149.0, 92.2)
- moved U4 0.75 mm to (142.1, 95.1)
- moved C3 0.71 mm to (153.0, 71.8)
- moved R13 0.50 mm to (163.0, 86.5)
- moved R7 0.50 mm to (158.2, 86.5)
Connections:
- C20 pad 1: HR_SIGNAL -> Net-(C20-Pad1)
- R11 pad 1: Net-(U6-OUT) -> Net-(JP1-A)
- R12 pad 2: Net-(U6-OUT) -> Net-(JP1-B)
- R13 pad 1: Net-(U5-*RESET) -> /LED_RST
- R24 pad 1: HR_SIGNAL -> Net-(C20-Pad1)
- TP3 pad 1: HR_SIGNAL -> Net-(C20-Pad1)
- U3 pad 15: unconnected-(U3-IO11-Pad15) -> /LED_RST
- U3 pad 27: /BACKLIGHT_EN -> unconnected-(U3-IO47-Pad27)
- U4 pad 1: HR_SIGNAL -> Net-(C20-Pad1)
- U4 pad 4: +3.3V -> Net-(JP3-B)
- U5 pad 25: Net-(U5-*RESET) -> /LED_RST
- U6 pad 1: Net-(U6-OUT) -> Net-(JP1-A)
- U6 pad 5: +3.3V -> VBUS
Routing:
- net /LED_RST: track 0.00 -> 36.8 mm, vias 0 -> 2
- net Net-(JP3-B): track 0.00 -> 13.7 mm, vias 0 -> 2
- net Net-(C20-Pad1): track 0.00 -> 12.3 mm
- net HR_SIGNAL: track 15.8 -> 3.95 mm
- net Net-(JP1-A): track 0.00 -> 9.94 mm
- net Net-(U6-OUT): track 9.59 -> 0.00 mm
- net VBUS: track 176.3 -> 182.8 mm, vias 5 -> 6
- net Net-(U5-*RESET): track 5.66 -> 0.00 mm
- net Net-(JP1-B): track 0.00 -> 3.59 mm
- net Net-(U4B-+): track 9.98 -> 8.48 mm
- net +3.3V: track 134.1 -> 132.9 mm, vias 9 -> 10
- net VCC/2: track 26.0 -> 25.2 mm
- net GND: vias 101 -> 741
