File: pulseoximeter.kicad_sch (KiCad schematic)
At the start: 45 parts, among them J1 X05A20L15T, J2 TYPE-C-31-M-12, J3 Conn_01x02, U1 TPD2EUSB30DRTR, U2 TPS7A4700RGWR, U3 ESP32-S3-MINI-1-N8, U4 LM324, U6 OPA140AIDBVR, U7 DMN2310UT-13

Commit message: layout complete
Parts:
- removed C18: 440pF, Capacitor_SMD:C_0603_1608Metric, symbol Device:C
- removed C6: 10uF, Capacitor_SMD:C_0603_1608Metric, symbol Device:C
- removed C7: 0.1uF, Capacitor_SMD:C_0603_1608Metric, symbol Device:C
- removed D2, D3: LED, LED_THT:LED_D3.0mm, symbol Device:LED
- removed R1: 10k, Resistor_SMD:R_0402_1005Metric, symbol Device:R
- removed R14, R22: 330, Resistor_SMD:R_0603_1608Metric, symbol Device:R
- removed R2: 1M, Resistor_SMD:R_0402_1005Metric, symbol Device:R
- removed U7: DMN2310UT-13, Package_TO_SOT_SMD:SOT-523, symbol 2N7002:2N7002
- added C8: 22uF, Capacitor_SMD:C_0603_1608Metric, symbol Device:C
- added D4, D7, D8, D9: LED, LED_THT:LED_D3.0mm, symbol Device:LED
- added TP3, TP4: TestPoint, TestPoint:TestPoint_Pad_D1.0mm, symbol Connector:TestPoint
- added U5: TLC59116IPWR, PW28, symbol TLC59116IPWR:TLC59116IPWR
- R11: value 8.1M -> 5.6M
- R13: value 330 -> 10k
- R7: value 330 -> 931
Connections:
- net +3.3V: now also R13.2, U4.4 (V+), U6.5 (V+), U5.28 (VCC)
- net DISPLAY_CLK: now also U3.20 (IO16); no longer U3.18 (IO14)
- net DISPLAY_CS: now also U3.21 (IO17); no longer U3.17 (IO13)
- net DISPLAY_D/C: now also U3.22 (IO18); no longer U3.16 (IO12)
- net DISPLAY_RESET: now also U3.18 (IO14); no longer U3.20 (IO16)
- net GND: now also R7.1, C8.2, U5.10 (GND), U5.19 (GND), U5.2 (A0), U5.24 (GND), U5.3 (A1), U5.4 (A2), U5.5 (A3); no longer D5.1 (K), D6.1 (K)
- net HR_SIGNAL: now also C8.1, TP3.1
- net LEDK: now also TP4.1, U5.22 (*OUT14)
- net SCL: now also U5.26 (SCL)
- net SDA: now also U5.27 (SDA)
- net TP_INT: now also U3.16 (IO12); no longer U3.22 (IO18)
- net TP_RST: now also U3.17 (IO13); no longer U3.21 (IO17)
- net VBUS: now also D5.2 (A), D6.2 (A), D4.2 (A), D7.2 (A), D8.2 (A), D9.2 (A); no longer R13.1, R7.1, U4.4 (V+), U6.5 (V+)
- net VCC/2: now also U4.13 (-); no longer U4.12 (+)
- net at R7.2: now also U5.1 (REXT); no longer D5.2 (A)
- net at R10.1, R9.2: now also U4.12 (+); no longer U4.13 (-)
- new net: D6.1 (K), U5.20 (*OUT12)
- new net: D7.1 (K), U5.6 (*OUT0)
- new net: D5.1 (K), U5.9 (*OUT3)
- new net: D9.1 (K), U5.15 (*OUT8)
- new net: D4.1 (K), U5.14 (*OUT7)
- new net: D8.1 (K), U5.23 (*OUT15)
- new net: R13.1, U5.25 (*RESET)
- no-connect marks 37 -> 46
Other:
- moved on the sheet: C20, J1, R10, R23, R24, R9, U4A, U4D, U4E

Commit message: -
Parts:
- removed C8: 22uF, Capacitor_SMD:C_0603_1608Metric, symbol Device:C
- added JP1, JP3: SolderJumper_2_Bridged, Jumper:SolderJumper-2_P1.3mm_Open_RoundedPad1.0x1.5mm, symbol Jumper:SolderJumper_2_Bridged
- added R1: 100k, Resistor_SMD:R_0603_1608Metric, symbol Device:R
- added R2: 50k, Resistor_SMD:R_0603_1608Metric, symbol Device:R
- added TP5: TestPoint, TestPoint:TestPoint_Pad_D1.0mm, symbol Connector:TestPoint
- C13: value 0.1uF -> 0.22uF
- C3: footprint Capacitor_SMD:C_0402_1005Metric -> Capacitor_SMD:C_0603_1608Metric
- R7: value 931 -> 910
Connections:
- net +3.3V: now also TP5.1; no longer U4.4 (V+), U6.5 (V+)
- net GND: now also R1.2
- net HR_SIGNAL: now also R1.1, R2.2; no longer C20.1, R24.1, TP3.1, U4.1
- net VBUS: now also U6.5 (V+), JP3.1 (A)
- net at R11.1, U6.1 (OUT): now also JP1.1 (A); no longer R12.2
- net LED_RST: now reaches U3.15 (IO11)
- net LED_RST: now also R13.1, U5.25 (*RESET)
- net BACKLIGHT_EN: no longer names the net of U3.27 (IO47)
- new net: JP3.2 (B), U4.4 (V+)
- new net: C20.1, R2.1, R24.1, TP3.1, U4.1
- new net: JP1.2 (B), R12.2
Other:
- moved on the sheet: C13, D1, R3
